Commit message: Fix Wheel order

File: int_brain_description/urdf/ros2_control_hardware.xacro (robot description, xacro)
@@ -9,4 +9,14 @@
             <param name="is_feedforward">$(arg is_feedforward)</param>
         </hardware>
+        <joint name="front_right_shaft_joint">
+            <command_interface name="velocity" />
+            <state_interface name="position" />
+            <state_interface name="velocity" />
+        </joint>
+        <joint name="rear_right_shaft_joint">
+            <command_interface name="velocity" />
+            <state_interface name="position" />
+            <state_interface name="velocity" />
+        </joint>
         <joint name="front_left_shaft_joint">
             <command_interface name="velocity" />
@@ -15,14 +25,4 @@
         </joint>
         <joint name="rear_left_shaft_joint">
-            <command_interface name="velocity" />
-            <state_interface name="position" />
-            <state_interface name="velocity" />
-        </joint>
-        <joint name="front_right_shaft_joint">
-            <command_interface name="velocity" />
-            <state_interface name="position" />
-            <state_interface name="velocity" />
-        </joint>
-        <joint name="rear_right_shaft_joint">
             <command_interface name="velocity" />
             <state_interface name="position" />
