Commit message: feat: Update int_brain_description and int_brain_system packages
- Added dependency on int_brain_hardware in package.xml of int_brain_description.
- Introduced a new link (pcb_link) and joint (pcb_joint) in the URDF file for the PCB component.
- Replaced the imu_calibrate executable with imu_feedback_node in CMakeLists.txt and updated installation targets.
- Increased the update rate for the controller manager in controllers.yaml.
- Added a new EKF configuration file (ekf.yaml) for robot localization.
- Updated pltjg_ctrl_dbg.xml for improved UI layout and plot configurations.
- Enhanced teleop_joy_params.yaml to include parameters for the new imu_feedback_node.
- Modified view.rviz to include visualization settings for the new pcb_link.
- Updated system.launch.py to include EKF node and remap topics for odometry.
- Added imu_feedback_node to teleop_joy.launch.py for feedback based on IMU data.
- Updated package.xml of int_brain_system to include additional dependencies for robot localization and control.
- Removed obsolete IMU calibration and covariance nodes from src directory.
- Implemented imu_feedback.cpp to provide haptic feedback based on IMU linear acceleration.

File: int_brain_description/urdf/int_brain.xacro (robot description, xacro)
@@ -36,9 +36,35 @@
     </collision>
   </link>
+  <link name="pcb_link">
+    <inertial>
+      <origin xyz="0 0 -0.001" rpy="0 0 0" />
+      <mass value="0.02" />
+      <inertia ixx="1e-05" iyy="1e-05" izz="1e-05" ixy="0.0" iyz="0.0" ixz="0.0" />
+    </inertial>
+    <visual>
+      <origin xyz="-0.1 0.06 -0.001" rpy="0 0 0" />
+      <geometry>
+        <mesh filename="file://$(find int_brain_description)/meshes/int-brain-pcb.dae"
+          scale="0.001 0.001 0.001" />
+      </geometry>
+    </visual>
+    <collision>
+      <origin xyz="-0.1 0.06 -0.001" rpy="0 0 0" />
+      <geometry>
+        <mesh filename="file://$(find int_brain_description)/meshes/int-brain-pcb.dae"
+          scale="0.001 0.001 0.001" />
+      </geometry>
+    </collision>
+  </link>
+  <joint name="pcb_joint" type="fixed">
+    <parent link="base_link" />
+    <child link="pcb_link" />
+    <origin xyz="0 0 0.01" rpy="0 0 0" />
+  </joint>
   <link name="imu_link" />
   <joint name="imu_joint" type="fixed">
-    <parent link="base_link" />
+    <parent link="pcb_link" />
     <child link="imu_link" />
-    <origin xyz="0 0 0.061" rpy="3.1414 0 1.5707" />
+    <origin xyz="-0.0118 -0.0127 0" rpy="0 3.1414 -1.5707" />
   </joint>
   <joint name="base_footprint_to_base_link" type="fixed">

Commit message: Fix pcb orientation and imu frame

File: int_brain_description/urdf/int_brain.xacro (robot description, xacro)
@@ -60,5 +60,5 @@
     <parent link="base_link" />
     <child link="pcb_link" />
-    <origin xyz="0 0 0.01" rpy="0 0 0" />
+    <origin xyz="0 0 0.01" rpy="0 0 3.1414" />
   </joint>
   <link name="imu_link" />
@@ -66,5 +66,5 @@
     <parent link="pcb_link" />
     <child link="imu_link" />
-    <origin xyz="-0.0118 -0.0127 0" rpy="0 3.1414 -1.5707" />
+    <origin xyz="-0.0072 -0.0123 0" rpy="0 3.1414 -1.5707" />
   </joint>
   <joint name="base_footprint_to_base_link" type="fixed">
